File: andino_hardware/circuitos/circuitos_robot/circuitos_robot.kicad_sch (KiCad schematic)
At the start: 8 parts, among them J1 Conn_01x06_Pin, J2 Conn_01x06_Pin, J3 Conn_01x08_Pin, M1 Stepper_Motor_unipolar_6pin, U1 RaspberryPi-CM3, U2 A4954, U3 Flir_LEPTON

Commit message: Progreso_30/10/25
Parts:
- removed M1: Stepper_Motor_unipolar_6pin, symbol Motor:Stepper_Motor_unipolar_6pin
- removed U1: RaspberryPi-CM3, symbol MCU_Module:RaspberryPi-CM3
- removed U2: A4954, Package_SO:TSSOP-16-1EP_4.4x5mm_P0.65mm_EP3x3mm, symbol Driver_Motor:A4954
- removed U3: Flir_LEPTON, symbol Sensor_Optical:Flir_LEPTON
- added J1, J2, J5, J6: Conn_01x02_Pin, symbol Connector:Conn_01x02_Pin
- added J3: Conn_01x03_Pin, symbol Connector:Conn_01x03_Pin
- added J4: Conn_01x04_Pin, symbol Connector:Conn_01x04_Pin
- added U2: L298N, Package_TO_SOT_THT:TO-220-15_P2.54x2.54mm_StaggerOdd_Lead4.58mm_Vertical, symbol Driver_Motor:L298N
- renumbered J3 to IMU, J1 to Motor_L, J2 to Motor_R
Connections:
- net GND: now reaches Motor_L.1 (Pin_1)
- net GND: now also IMU.2 (Pin_2), Motor_R.1 (Pin_1), J3.2 (Pin_2)
- net Encoder_L_pinB: now reaches Motor_L.2 (Pin_2)
- net Encoder_L_pinB: now also A1.22 (A3)
- net Encoder_L_pinA: now reaches Motor_L.3 (Pin_3)
- net Encoder_L_pinA: now also A1.21 (A2)
- net 5V: now reaches Motor_L.4 (Pin_4)
- net 5V: now also IMU.1 (Pin_1), Motor_R.4 (Pin_4), J3.1 (Pin_1)
- net Motor_driver_L_pin2: now reaches Motor_L.5 (Pin_5)
- net Motor_driver_L_pin2: now also J2.2 (Pin_2)
- net Motor_driver_L_pin1: now reaches Motor_L.6 (Pin_6)
- net Motor_driver_L_pin1: now also J2.1 (Pin_1)
- net SCL: now reaches IMU.3 (Pin_3)
- net SCL: now also A1.24 (SCL/A5)
- net SDA: now reaches IMU.4 (Pin_4)
- net SDA: now also A1.23 (SDA/A4)
- net I2C: now reaches IMU.5 (Pin_5)
- net Interrup_pin: now reaches IMU.6 (Pin_6)
- net Flash: now reaches IMU.7 (Pin_7)
- net RST: now reaches IMU.8 (Pin_8)
- net PWM2: now reaches A1.12 (D9)
- net PWM2: now also J4.3 (Pin_3)
- net PWM4: now reaches A1.13 (D10)
- net PWM4: now also J4.1 (Pin_1)
- net PWM5: now reaches A1.15 (MISO)
- net SCK: now reaches A1.16 (SCK)
- net Encoder_R_pinA: now reaches A1.5 (D2)
- net Encoder_R_pinA: now also Motor_R.3 (Pin_3)
- net Encoder_R_pinB: now reaches A1.6 (D3)
- net Encoder_R_pinB: now also Motor_R.2 (Pin_2)
- net PWM1: now reaches A1.8 (D5)
- net PWM1: now also J4.4 (Pin_4)
- net PWM3: now reaches A1.9 (D6)
- net PWM3: now also J4.2 (Pin_2)
- net Motor_driver_R_pin2: now reaches Motor_R.5 (Pin_5)
- net Motor_driver_R_pin2: now also J1.1 (Pin_1)
- net Motor_driver_R_pin1: now reaches Motor_R.6 (Pin_6)
- net Motor_driver_R_pin1: now also J1.2 (Pin_2)
- new net 9V: J3.3 (Pin_3)
Other:
- note added: "Puente H"
- note added: "step up"
- moved on the sheet: A1, IMU, Motor_L, Motor_R
