File: andino_hardware/circuitos/Placa_1/circuitos_robot.kicad_sch (KiCad schematic)
At the start: 18 parts, among them J8 Jack-DC, SW1 Conn_01x03_Pin

Commit message: Primera placa impresa
Connections:
- net 12V_Fuente: now also J8.1; no longer J8.2
- net GND: now also A1.29 (GND), A1.4 (GND), J8.2, USB_Alimentacion1.5 (Shield), USB_Lidar1.5 (Shield), USB_RPI1.5 (Shield); no longer J8.1
- net PWM2: now also Puente_H1.2 (Pin_2); no longer Puente_H1.3 (Pin_3)
- net PWM3: now also Puente_H1.3 (Pin_3); no longer Puente_H1.2 (Pin_2)
- net D-: now reaches USB_Lidar1.2 (D-), USB_RPI1.2 (D-)
- net D+: now reaches USB_Lidar1.3 (D+), USB_RPI1.3 (D+)
Other:
- moved on the sheet: J8
