File: andino_hardware/circuitos/Placa_2/circuitos_robot.kicad_pcb (KiCad board)
At the start: 2 copper layers, 100 x 80 mm, 19 parts

Commit message: placa
Parts:
- removed G***: LOGO, LOGO
- removed USB: USB3_A_Molex_48393-001, Connector_USB:USB3_A_Molex_48393-001
- added C1: CP_Radial_D8.0mm_P3.80mm, Capacitor_THT:CP_Radial_D8.0mm_P3.80mm, F.Cu at (98.3, 33.7)
- added REF**: Regulador_RPI, Library_gero:Regulador_RPI, F.Cu at (92.4, 45.1)
- A1: renamed from Arduino NANO
- J8: renamed from Jack DC
- moved A1 59.6 mm to (61.4, 90.2), turned to 180 degrees
- moved Stepdown_LM2596 55.9 mm to (67.5, 41.7), turned to 180 degrees
- moved Motor_R1 54.9 mm to (67.8, 76.2), turned to 0 degrees
- moved USB_Lidar1 47.1 mm to (100.4, 79.6), turned to 180 degrees
- moved USB_RPI1 33.4 mm to (114.3, 81.7), turned to 90 degrees
- moved REF** 32.8 mm to (145.9, 84.8)
- moved G.F. 24.5 mm to (50.0, 3.35)
- moved D1 22.5 mm to (68.7, 97.7)
- moved Regulador_LIDAR 21.5 mm to (71.1, 24.4), turned to 0 degrees
- moved IMU1 16.4 mm to (35.4, 64.7)
- moved Puente_H1 11.0 mm to (67.9, 64.7), turned to 0 degrees
- moved Motor_L1 9.05 mm to (41.7, 72.4), turned to 180 degrees
- moved PH_V1 8.25 mm to (29.9, 50.5), turned to -90 degrees
- moved J8 5.32 mm to (109.3, 95.3)
- moved D2 3.64 mm to (89.0, 97.6)
- renumbered Baterias to Baterias1, IMU to IMU1, Motor_L to Motor_L1, Motor_R to Motor_R1, PH_V to PH_V1, Puente_H to Puente_H1, Regulador_USB to Regulador_LIDAR, SW to SW1, USB to USB_Lidar1, USB to USB_RPI1
Connections:
- A1 pad 30: 9V -> unconnected-(A1-VIN-Pad30)
Routing:
- net GND: track 797.1 -> 227.6 mm
- net 12V: track 145.4 -> 7.41 mm
- net 9V: track 112.5 -> 16.7 mm
- net Encoder_R_pinA: track 92.4 -> 6.97 mm
- net Encoder_R_pinB: track 89.1 -> 6.97 mm
- net Encoder_L_pinB: track 67.6 -> 4.47 mm
- net SDA: track 76.5 -> 13.5 mm
- net Encoder_L_pinA: track 63.8 -> 4.47 mm
- net 5V_Ard: track 155.3 -> 100.5 mm
- net SCL: track 80.4 -> 32.5 mm
- net 5V: track 51.6 -> 15.9 mm
- net D+: track 35.0 -> 0.00 mm
- net D-: track 34.3 -> 0.00 mm
- net Net-(D1-A): track 20.5 -> 0.00 mm
- net PWM1: track 26.3 -> 6.53 mm
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- removed copper zone on B.Cu, net GND
Other:
- board text removed: "Alimentación"
