File: andino_hardware/circuitos/Placa_2/circuitos_robot.kicad_pcb (KiCad board)
At the start: 2 copper layers, 100 x 80 mm, 19 parts, among them J8 Jack-DC, SW1 Conn_01x03_Pin

Commit message: camara funciona
Parts:
- removed Regulador_LIDAR: Regulador_USB, Library_gero:Regulador_USB
- removed SW1: Conn_01x03_Pin, Connector_Wire:SolderWire-0.5sqmm_1x03_P4.8mm_D0.9mm_OD2.3mm
- added REF**: MountingHole_3.2mm_M3, MountingHole:MountingHole_3.2mm_M3, F.Cu at (38.6, 79.6)
- added REF**: Regulador_USB, Library_gero:Regulador_USB, F.Cu at (71.1, 22.1)
- added sw: Conn_01x02_Pin, Connector_Wire:SolderWire-0.1sqmm_1x02_P3.6mm_D0.4mm_OD1mm, F.Cu at (38.4, 96.9)
- Alimentación RPI: renamed from REF**
- moved G.F. 73.2 mm to (120.2, 24.0)
- moved C1 48.6 mm to (97.6, 82.3), turned to 180 degrees
- moved REF** 25.7 mm to (120.2, 85.0)
- moved D1 21.2 mm to (89.7, 94.6), turned to 0 degrees
- moved D2 8.72 mm to (89.7, 88.9)
- moved USB_RPI1 3.57 mm to (112.3, 78.7)
- moved USB_Lidar1 3.25 mm to (99.3, 76.6)
- moved IMU1 2.76 mm to (32.6, 64.4)
- moved Motor_L1 1.30 mm to (40.4, 72.3)
- moved Motor_R1 1.11 mm to (66.8, 75.8)
- moved Alimentación RPI 1.10 mm to (91.3, 45.2)
- moved Puente_H1 0.81 mm to (67.9, 63.9)
- moved J8 0.49 mm to (109.8, 95.5)
- moved PH_V1 0.25 mm to (29.7, 50.5)
Routing:
- net 12V: track 7.41 -> 154.3 mm
- net GND: track 227.6 -> 348.0 mm, vias 0 -> 2
- net Net-(D1-A): track 0.00 -> 65.6 mm
- net 5V: track 15.9 -> 68.7 mm
- net D+: track 0.00 -> 48.6 mm
- net D-: track 0.00 -> 37.1 mm
- net 5V_Ard: track 100.5 -> 112.5 mm
- net 12V_Bateria: track 17.0 -> 5.35 mm
- net 12V_Fuente: track 0.00 -> 9.91 mm
- net SCL: track 32.5 -> 40.3 mm
- net Encoder_L_pinA: track 4.47 -> 5.77 mm
- net Encoder_L_pinB: track 4.47 -> 5.77 mm
- net Encoder_R_pinB: track 6.97 -> 5.77 mm
- net Encoder_R_pinA: track 6.97 -> 5.77 mm
- net PWM4: track 8.60 -> 9.26 mm
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- added copper zone on B.Cu, net 12V
- added copper zone on B.Cu, net 5V_Ard
- added copper zone on B.Cu, net GND
Other:
- board text added: "interruptor chico"
- board text removed: "-"
- board text removed: "Lidar"
- board text removed: "RPI"
