File: andino_hardware/circuitos/Placa_2/circuitos_robot.kicad_sch (KiCad schematic)
At the start: 18 parts, among them J8 Jack-DC, SW1 Conn_01x03_Pin

Commit message: placa
Parts:
- removed Reg_USB_IN1, Reg_USB_OUT1, Step_up_IN1, Step_up_OUT1: Conn_01x02_Pin, Connector_Wire:SolderWire-0.1sqmm_1x02_P3.6mm_D0.4mm_OD1mm, symbol Connector:Conn_01x02_Pin
- removed USB_Alimentacion1: USB_A, Connector_USB:USB_A_CONNFLY_DS1095-WNR0, symbol Connector:USB_A
Connections:
- net 9V: no longer A1.30 (VIN)
Other:
- note removed: "USB"
