File: andino_hardware/circuitos/Placa_3/circuitos_robot.kicad_pcb (KiCad board)
At the start: 2 copper layers, 100 x 80 mm, 20 parts, among them J8 Jack-DC

Commit message: placa lista
Parts:
- removed G.F.: MountingHole_3.2mm_M3, MountingHole:MountingHole_3.2mm_M3
- Regulador USB: renamed from REF**
- moved Motor_L 136.3 mm to (68.0, 35.8)
- moved PH_PWM 120.6 mm to (79.4, 64.8)
- moved Motor_R 120.3 mm to (65.4, 64.8)
- moved PH_V 107.1 mm to (29.2, 59.0)
- moved REF** 78.0 mm to (33.9, 36.5)
- moved REF** 73.6 mm to (103.2, 46.9)
- moved IMU 20.1 mm to (41.0, 45.0), turned to 180 degrees
- moved Arduino_NANO 11.1 mm to (50.2, 58.3)
- moved J8 9.74 mm to (113.1, 86.3), turned to 0 degrees
- moved C1 8.45 mm to (102.5, 61.1)
- moved Stepdown_LM2596 4.83 mm to (70.3, 90.5)
- moved Regulador USB 4.39 mm to (75.5, 71.2)
- moved Bat 4.24 mm to (32.2, 92.8), turned to -90 degrees
- moved USB_RPI 1.59 mm to (107.1, 73.8)
- moved D1 0.83 mm to (81.1, 95.5)
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- renumbered A1 to Arduino_NANO, Baterias1 to Bat, IMU1 to IMU, Motor_L1 to Motor_L, Motor_R1 to Motor_R, Puente_H1 to PH_PWM, PH_V1 to PH_V, SW_17,2*7,6 to SW, USB_Lidar1 to USB_Lidar, USB_RPI1 to USB_RPI
Connections:
- SW pad 4: (no net) -> GND
Routing:
- net 5V_Ard: track 0.00 -> 125.8 mm
- net 5V: track 0.00 -> 55.8 mm
- net 12V: track 0.00 -> 55.5 mm
- net 9V: track 0.00 -> 49.2 mm
- net D+: track 0.00 -> 40.8 mm
- net D-: track 0.00 -> 36.4 mm
- net SDA: track 0.00 -> 31.0 mm
- net SCL: track 0.00 -> 27.5 mm
- net 12V_Bateria: track 0.00 -> 21.0 mm
- net Net-(D1-A): track 0.00 -> 18.4 mm
- net 12V_Fuente: track 0.00 -> 16.2 mm
- net PWM3: track 0.00 -> 9.33 mm
- net PWM1: track 0.00 -> 8.78 mm
- net Encoder_L_pinB: track 0.00 -> 7.29 mm
- net Encoder_L_pinA: track 0.00 -> 7.29 mm
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- added copper zone on B.Cu, net 12V
- added copper zone on B.Cu, net GND
Other:
- board text added: "Andino"
- board text removed: "interruptor chico"

Commit message: impresion de pcb
Parts:
- removed the Bat at (32.2, 92.8)
- removed the PH_V at (29.2, 59.0)
- added ?: , clipboard:e55b3b5e-7304-4eca-bfe6-4dad5b5e2501, F.Cu at (59.4, 28.3)
- added Bat: PinHeader_1x02_P2.54mm_Vertical, Connector_PinHeader_2.54mm:PinHeader_1x02_P2.54mm_Vertical, F.Cu at (34.5, 96.0)
- added PH_V: PinHeader_1x02_P2.54mm_Vertical, Connector_PinHeader_2.54mm:PinHeader_1x02_P2.54mm_Vertical, F.Cu at (29.3, 55.6)
- renumbered Motor_R to Motor_L, Motor_L to Motor_R
Routing:
- net 9V: track 49.2 -> 45.8 mm
- net 5V_Ard: track 125.8 -> 123.0 mm
- net 12V_Bateria: track 21.0 -> 21.5 mm
